File: SplitFlapDriverATtiny1616 V2/SplitFlapDriverATtiny1616V2.kicad_pcb (KiCad board)
At the start: 2 copper layers, 30 x 60 mm, 25 parts, among them J1 UPDI Programming, J2 Conn_01x01_Pin, J3 Stepper Connector, J4 Hall Effect, J5 Conn_01x05_Pin, J6 Conn_01x01_Pin, J7 Conn_01x01_Pin, J8 Conn_01x01_Pin, U1 ATtiny1616-MNR, U2 ULN2003ADR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

Commit message: Updated Hall Effect Header to JST-PH
Parts:
- J4: footprint Connector_PinHeader_2.54mm:PinHeader_1x03_P2.54mm_Vertical -> Connector_JST:JST_PH_B3B-PH-K_1x03_P2.00mm_Vertical
- moved J4 19.7 mm to (128.2, 103.5)
- moved C3 8.42 mm to (125.6, 120.9)
- moved C4 8.42 mm to (127.1, 120.9)
- moved C7 8.42 mm to (128.6, 120.9)
- moved C8 8.42 mm to (129.5, 114.6)
- moved U5 8.42 mm to (127.1, 109.7)
- moved C5 8.42 mm to (124.6, 109.8)
- moved C6 8.42 mm to (129.6, 109.7)
- moved C9 8.42 mm to (124.6, 114.6)
- moved R1 8.42 mm to (128.0, 118.2)
- moved U6 8.42 mm to (127.1, 114.6)
Routing:
- net HALL_IN: track 42.0 -> 12.4 mm, vias 2 -> 0
- net +3V3: track 27.2 -> 37.6 mm
- net +VBUS: track 13.3 -> 21.7 mm
- net RS465_A: track 26.1 -> 30.2 mm
- net +5V: track 22.9 -> 19.0 mm
- net GND: track 23.0 -> 26.1 mm, vias 15 -> 16
- net +VBUSF: track 45.4 -> 47.1 mm
