File: SplitFlapDriverATtiny1616 V2/SplitFlapDriverATtiny1616V2.kicad_sch (KiCad schematic)
At the start: 25 parts, among them J1 UPDI Programming, J2 Conn_01x01_Pin, J3 Stepper Connector, J4 Hall Effect, J5 Conn_01x05_Pin, J6 Conn_01x01_Pin, J7 Conn_01x01_Pin, J8 Conn_01x01_Pin, U1 ATtiny1616-MNR, U2 ULN2003ADR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

Commit message: Updated Hall Effect Header to JST-PH
Parts:
- J4: footprint Connector_PinHeader_2.54mm:PinHeader_1x03_P2.54mm_Vertical -> Connector_JST:JST_PH_B3B-PH-K_1x03_P2.00mm_Vertical
Changed lines of the file:
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@@
 			)
 		)
-		(property "Footprint" "Connector_PinHeader_2.54mm:PinHeader_1x03_P2.54mm_Vertical"
+		(property "Footprint" "Connector_JST:JST_PH_B3B-PH-K_1x03_P2.00mm_Vertical"
 			(at 91.44 153.67 0)
 			(effects
